Commit message: wednesday lab changes - preparing for SLAM setup

File: install/r2d10/share/r2d10/urdf/assembly_3.urdf (robot description, URDF)
Before this commit: robot assembly_3, 8 links, 7 joints
Joints:
- removed joint Revolute 2
- removed joint Revolute 3
- removed joint Rigid 1
- removed joint Rigid 5
- removed joint Rigid 6
- removed joint Rigid 7
- removed joint Rigid 9
- added joint Revolute_2: type continuous, parent base_link, child left_wheel_1, origin xyz=-0.085 -0.0475 0.02 rpy=0 0 0, axis -1.0 0.0 0.0
- added joint Revolute_3: type continuous, parent base_link, child right_wheel_1, origin xyz=0.09 -0.0475 0.02 rpy=0 0 0, axis -1.0 0.0 0.0
- added joint Rigid_1: type fixed, parent base_link, child caster_1, origin xyz=0.0 0.0 0.0 rpy=0 0 0
- added joint Rigid_5: type fixed, parent base_link, child ultrasonic_forward_1, origin xyz=0.0 0.15 0.035 rpy=0 0 0
- added joint Rigid_6: type fixed, parent base_link, child ultrasonic_left_1, origin xyz=-0.15 0.0 0.035 rpy=0 0 0
- added joint Rigid_7: type fixed, parent base_link, child ultrasonic_right_1, origin xyz=0.15 0.0 0.035 rpy=0 0 0
- added joint Rigid_9: type fixed, parent base_link, child lidar_1, origin xyz=0.0 0.0 0.07 rpy=0 0 0

Commit message: changes to run SLAM

File: install/r2d10/share/r2d10/urdf/assembly_3.urdf (robot description, URDF)
Before this commit: robot assembly_3, 8 links, 7 joints
Links:
- added link chassis, mass 37.821366170820795; collision mesh filename=package://r2d10/meshes/base_link.stl scale=0.001 0.001 0.001; visual mesh filename=package://r2d10/meshes/base_link.stl scale=0.001 0.001 0.001
- added link imu_link
- link base_link: mass 37.821366170820795 -> None; geometry 
Joints:
- removed joint Revolute_2
- removed joint Revolute_3
- removed joint Rigid_1
- removed joint Rigid_5
- removed joint Rigid_6
- removed joint Rigid_7
- removed joint Rigid_9
- added joint caster_joint: type fixed, parent chassis, child caster_1, origin xyz=0.0 0.0 0.0 rpy=0 0 0
- added joint chassis_joint: type fixed, parent base_link, child chassis, origin xyz=0 0 0 rpy=0 0 0
- added joint imu_joint: type fixed, parent base_link, child imu_link, origin xyz=0 0 0 rpy=0 0 0
- added joint left_wheel_joint: type continuous, parent base_link, child left_wheel_1, origin xyz=-0.085 -0.0475 0.02 rpy=0 0 0, axis -1.0 0.0 0.0
- added joint lidar_joint: type fixed, parent chassis, child lidar_1, origin xyz=0.0 0.0 0.07 rpy=0 0 0
- added joint right_wheel_joint: type continuous, parent base_link, child right_wheel_1, origin xyz=0.09 -0.0475 0.02 rpy=0 0 0, axis -1.0 0.0 0.0
- added joint ultrasonic_forward_joint: type fixed, parent chassis, child ultrasonic_forward_1, origin xyz=0.0 0.15 0.035 rpy=0 0 0
- added joint ultrasonic_left_joint: type fixed, parent chassis, child ultrasonic_left_1, origin xyz=-0.15 0.0 0.035 rpy=0 0 0
- added joint ultrasonic_right_joint: type fixed, parent chassis, child ultrasonic_right_1, origin xyz=0.15 0.0 0.035 rpy=0 0 0

File: install/r2d10/share/r2d10/urdf/assembly_3.urdf.xacro (robot description, xacro)
@@ -1,212 +1,249 @@
 <?xml version="1.0"?>
 <robot name="assembly_3" xmlns:xacro="http://www.ros.org/wiki/xacro">
-<!-- <xacro:include filename="$(find r2d10)/urdf/materials.xacro"/> -->
-<!-- <xacro:include filename="$(find-pkg-share r2d10)/urdf/assembly_3.trans"/>
-<xacro:include filename="$(find-pkg-share r2d10)/urdf/assembly_3.gazebo"/> -->
-<material name="silver"> <!-- colour is silver -->
-  <color rgba="0.700 0.700 0.700 1.000"/>
-</material>
-<material name="black"> <!-- wheels colour black -->
-  <color rgba="0 0 0 1"/>
-</material>
-<!-- physical part base_link -->
-<link name="base_link">
-  <inertial>   <!-- inertia link -->
-    <origin xyz="-6.745525765719935e-05 0.0012816498954868177 0.0354047315459432" rpy="0 0 0"/>  <!-- position & rotation -->
-    <mass value="37.821366170820795"/> <!-- mass (kg) -->
-    <inertia ixx="0.23125" iyy="0.223709" izz="0.423982" ixy="-0.000124" iyz="0.000747" ixz="-3.9e-05"/>  <!-- inertia matrix -->
-  </inertial>
-  <visual>
-    <origin xyz="0 0 0" rpy="0 0 0"/> <!-- position and rotation -->
-    <geometry>
-      <mesh filename="package://r2d10/meshes/base_link.stl" scale="0.001 0.001 0.001"/>
-    </geometry>
-    <material name="silver"/>
-  </visual>
-  <collision> <!-- physics collision shape -->
-    <origin xyz="0 0 0" rpy="0 0 0"/>
-    <geometry> <!-- shape of visual collision -->
-      <mesh filename="package://r2d10/meshes/base_link.stl" scale="0.001 0.001 0.001"/>
-    </geometry>
-  </collision>
-</link>
-<!-- link: physical part caster_1 -->
-<link name="caster_1">
-  <inertial>
-    <origin xyz="0.0 0.11 -0.0043996518255540636" rpy="0 0 0"/>
-    <mass value="0.0707011858312227"/>
-    <inertia ixx="6e-06" iyy="6e-06" izz="1e-05" ixy="0.0" iyz="-0.0" ixz="0.0"/>
-  </inertial>
-  <visual>
-    <origin xyz="-0.0 -0.0 -0.0" rpy="0 0 0"/>
-    <geometry>
-      <mesh filename="package://r2d10/meshes/caster_1.stl" scale="0.001 0.001 0.001"/>
-    </geometry>
-    <material name="silver"/>
-  </visual>
-  <collision>
-    <origin xyz="-0.0 -0.0 -0.0" rpy="0 0 0"/>
-    <geometry>
-      <mesh filename="package://r2d10/meshes/caster_1.stl" scale="0.001 0.001 0.001"/>
-    </geometry>
-  </collision>
-</link>
-<link name="left_wheel_1">
-  <inertial>
-    <origin xyz="-0.012500000000000011 0.0 0.0" rpy="0 0 0"/>
-    <mass value="0.6512177959195155"/>
-    <inertia ixx="0.000344" iyy="0.000206" izz="0.000206" ixy="0.0" iyz="-0.0" ixz="0.0"/>
-  </inertial>
-  <visual>
-    <origin xyz="0.085 0.0475 -0.02" rpy="0 0 0"/>
-    <geometry>
-      <mesh filename="package://r2d10/meshes/left_wheel_1.stl" scale="0.001 0.001 0.001"/>
-    </geometry>
-    <material name="black"/>
-  </visual>
-  <collision>
-    <origin xyz="0.085 0.0475 -0.02" rpy="0 0 0"/>
-    <geometry>
-      <mesh filename="package://r2d10/meshes/left_wheel_1.stl" scale="0.001 0.001 0.001"/>
-    </geometry>
-  </collision>
-</link>
-<link name="right_wheel_1">
-  <inertial>
-    <origin xyz="0.012500000000000108 0.0 -6.938893903907228e-18" rpy="0 0 0"/>
-    <mass value="0.6512177959195155"/>
-    <inertia ixx="0.000344" iyy="0.000206" izz="0.000206" ixy="0.0" iyz="0.0" ixz="0.0"/>
-  </inertial>
-  <visual>
-    <origin xyz="-0.09 0.0475 -0.02" rpy="0 0 0"/>
-    <geometry>
-      <mesh filename="package://r2d10/meshes/right_wheel_1.stl" scale="0.001 0.001 0.001"/>
-    </geometry>
-    <material name="black"/>
-  </visual>
-  <collision>
-    <origin xyz="-0.09 0.0475 -0.02" rpy="0 0 0"/>
-    <geometry>
-      <mesh filename="package://r2d10/meshes/right_wheel_1.stl" scale="0.001 0.001 0.001"/>
-    </geometry>
-  </collision>
-</link>
-<link name="ultrasonic_forward_1">
-  <inertial>
-    <origin xyz="-6.89984745874354e-13 0.005799256348663379 -6.55503359925369e-11" rpy="0 0 0"/>
-    <mass value="0.06306919012201337"/>
-    <inertia ixx="3e-06" iyy="1.2e-05" izz="1.2e-05" ixy="-0.0" iyz="0.0" ixz="-0.0"/>
-  </inertial>
-  <visual>
-    <origin xyz="-0.0 -0.15 -0.035" rpy="0 0 0"/>
-    <geometry>
-      <mesh filename="package://r2d10/meshes/ultrasonic_forward_1.stl" scale="0.001 0.001 0.001"/>
-    </geometry>
-    <material name="silver"/>
-  </visual>
-  <collision>
-    <origin xyz="-0.0 -0.15 -0.035" rpy="0 0 0"/>
-    <geometry>
-      <mesh filename="package://r2d10/meshes/ultrasonic_forward_1.stl" scale="0.001 0.001 0.001"/>
-    </geometry>
-  </collision>
-</link>
-<link name="ultrasonic_left_1">
-  <inertial>
-    <origin xyz="-0.005799256348663379 -6.899762237296075e-13 -6.55503359925369e-11" rpy="0 0 0"/>
-    <mass value="0.06306919012201337"/>
-    <inertia ixx="1.2e-05" iyy="3e-06" izz="1.2e-05" ixy="0.0" iyz="-0.0" ixz="-0.0"/>
-  </inertial>
-  <visual>
-    <origin xyz="0.15 -0.0 -0.035" rpy="0 0 0"/>
-    <geometry>
-      <mesh filename="package://r2d10/meshes/ultrasonic_left_1.stl" scale="0.001 0.001 0.001"/>
-    </geometry>
-    <material name="silver"/>
-  </visual>
-  <collision>
-    <origin xyz="0.15 -0.0 -0.035" rpy="0 0 0"/>
-    <geometry>
-      <mesh filename="package://r2d10/meshes/ultrasonic_left_1.stl" scale="0.001 0.001 0.001"/>
-    </geometry>
-  </collision>
-</link>
-<link name="ultrasonic_right_1">
-  <inertial>
-    <origin xyz="0.005799256348663379 6.899932680191004e-13 -6.55503359925369e-11" rpy="0 0 0"/>
-    <mass value="0.06306919012201337"/>
-    <inertia ixx="1.2e-05" iyy="3e-06" izz="1.2e-05" ixy="0.0" iyz="0.0" ixz="0.0"/>
-  </inertial>
-  <visual>
-    <origin xyz="-0.15 -0.0 -0.035" rpy="0 0 0"/>
-    <geometry>
-      <mesh filename="package://r2d10/meshes/ultrasonic_right_1.stl" scale="0.001 0.001 0.001"/>
-    </geometry>
-    <material name="silver"/>
-  </visual>
-  <collision>
-    <origin xyz="-0.15 -0.0 -0.035" rpy="0 0 0"/>
-    <geometry>
-      <mesh filename="package://r2d10/meshes/ultrasonic_right_1.stl" scale="0.001 0.001 0.001"/>
-    </geometry>
-  </collision>
-</link>
-<link name="lidar_1">
-  <inertial>
-    <origin xyz="7.385233546074017e-18 0.0 0.01999999999999999" rpy="0 0 0"/>
-    <mass value="1.2084136142033137"/>
-    <inertia ixx="0.000531" iyy="0.000531" izz="0.00074" ixy="0.0" iyz="0.0" ixz="0.0"/>
-  </inertial>
-  <visual>
-    <origin xyz="-0.0 -0.0 -0.07" rpy="0 0 0"/>
-    <geometry>
-      <mesh filename="package://r2d10/meshes/lidar_1.stl" scale="0.001 0.001 0.001"/>
-    </geometry>
-    <material name="silver"/>
-  </visual>
-  <collision>
-    <origin xyz="-0.0 -0.0 -0.07" rpy="0 0 0"/>
-    <geometry>
-      <mesh filename="package://r2d10/meshes/lidar_1.stl" scale="0.001 0.001 0.001"/>
-    </geometry>
-  </collision>
-</link>
-<!-- joint part connectors such as type and name -->
-<joint name="Rigid 1" type="fixed">
-  <origin xyz="0.0 0.0 0.0" rpy="0 0 0"/>
-  <parent link="base_link"/>
-  <child link="caster_1"/>
-</joint>
-<joint name="Revolute 2" type="continuous">
-  <origin xyz="-0.085 -0.0475 0.02" rpy="0 0 0"/>
-  <parent link="base_link"/>
-  <child link="left_wheel_1"/>
-  <axis xyz="-1.0 0.0 0.0"/>
-</joint>
-<joint name="Revolute 3" type="continuous">
-  <origin xyz="0.09 -0.0475 0.02" rpy="0 0 0"/>
-  <parent link="base_link"/>
-  <child link="right_wheel_1"/>
-  <axis xyz="1.0 0.0 0.0"/>
-</joint>
-<joint name="Rigid 5" type="fixed">
-  <origin xyz="0.0 0.15 0.035" rpy="0 0 0"/>
-  <parent link="base_link"/>
-  <child link="ultrasonic_forward_1"/>
-</joint>
-<joint name="Rigid 6" type="fixed">
-  <origin xyz="-0.15 0.0 0.035" rpy="0 0 0"/>
-  <parent link="base_link"/>
-  <child link="ultrasonic_left_1"/>
-</joint>
-<joint name="Rigid 7" type="fixed">
-  <origin xyz="0.15 0.0 0.035" rpy="0 0 0"/>
-  <parent link="base_link"/>
-  <child link="ultrasonic_right_1"/>
-</joint>
-<joint name="Rigid 9" type="fixed">
-  <origin xyz="0.0 0.0 0.07" rpy="0 0 0"/>
-  <parent link="base_link"/>
-  <child link="lidar_1"/>
-</joint>
+    <xacro:include filename="$(find r2d10)/urdf/r2d10.gazebo" />
+    <xacro:include filename="$(find r2d10)/urdf/inertial_macros.xacro" />
+    <!-- MATERIALS -->
+    <material name="silver">
+        <color rgba="0.700 0.700 0.700 1.000"/>
+    </material>
+    <material name="black">
+        <color rgba="0 0 0 1"/>
+    </material>
+    <!-- BASE LINK -->
+    <link name="base_link">
+    </link>
+    <!-- CHASSIS (your base_link visual/collision) -->
+    <joint name="chassis_joint" type="fixed">
+        <parent link="base_link"/>
+        <child link="chassis"/>
+        <origin xyz="0 0 0" rpy="0 0 0"/>
+    </joint>
+    <link name="chassis">
+        <inertial>
+            <origin xyz="-6.745525765719935e-05 0.0012816498954868177 0.0354047315459432" rpy="0 0 0"/>
+            <mass value="37.821366170820795"/>
+            <inertia ixx="0.23125" iyy="0.223709" izz="0.423982" ixy="-0.000124" iyz="0.000747" ixz="-3.9e-05"/>
+        </inertial>
+        <visual>
+            <origin xyz="0 0 0" rpy="0 0 0"/>
+            <geometry>
+                <mesh filename="file://$(find r2d10)/meshes/base_link.stl" scale="0.001 0.001 0.001"/>
+            </geometry>
+            <material name="silver"/>
+        </visual>
+        <collision>
+            <origin xyz="0 0 0" rpy="0 0 0"/>
+            <geometry>
+                <mesh filename="file://$(find r2d10)/meshes/base_link.stl" scale="0.001 0.001 0.001"/>
+            </geometry>
+        </collision>
+    </link>
+    <!-- CASTER LINK -->
+    <joint name="caster_joint" type="fixed">
+        <origin xyz="0.0 0.0 0.0" rpy="0 0 0"/>
+        <parent link="chassis"/>
+        <child link="caster_1"/>
+    </joint>
+    <link name="caster_1">
+        <inertial>
+            <origin xyz="0.0 0.11 -0.0043996518255540636" rpy="0 0 0"/>
+            <mass value="0.0707011858312227"/>
+            <inertia ixx="6e-06" iyy="6e-06" izz="1e-05" ixy="0.0" iyz="-0.0" ixz="0.0"/>
+        </inertial>
+        <visual>
+            <origin xyz="-0.0 -0.0 -0.0" rpy="0 0 0"/>
+            <geometry>
+                <mesh filename="file://$(find r2d10)/meshes/caster_1.stl" scale="0.001 0.001 0.001"/>
+            </geometry>
+            <material name="silver"/>
+        </visual>
+        <collision>
+            <origin xyz="-0.0 -0.0 -0.0" rpy="0 0 0"/>
+            <geometry>
+                <mesh filename="file://$(find r2d10)/meshes/caster_1.stl" scale="0.001 0.001 0.001"/>
+            </geometry>
+        </collision>
+    </link>
+    <!-- LEFT WHEEL LINK -->
+    <joint name="left_wheel_joint" type="continuous">
+        <origin xyz="-0.085 -0.0475 0.02" rpy="0 0 0"/>
+        <parent link="base_link"/>
+        <child link="left_wheel_1"/>
+        <axis xyz="-1.0 0.0 0.0"/>
+    </joint>
+    <link name="left_wheel_1">
+        <inertial>
+            <origin xyz="-0.012500000000000011 0.0 0.0" rpy="0 0 0"/>
+            <mass value="0.6512177959195155"/>
+            <inertia ixx="0.000344" iyy="0.000206" izz="0.000206" ixy="0.0" iyz="-0.0" ixz="0.0"/>
+        </inertial>
+        <visual>
+            <origin xyz="0.085 0.0475 -0.02" rpy="0 0 0"/>
+            <geometry>
+                <mesh filename="file://$(find r2d10)/meshes/left_wheel_1.stl" scale="0.001 0.001 0.001"/>
+            </geometry>
+            <material name="black"/>
+        </visual>
+        <collision>
+            <origin xyz="0.085 0.0475 -0.02" rpy="0 0 0"/>
+            <geometry>
+               <mesh filename="file://$(find r2d10)/meshes/left_wheel_1.stl" scale="0.001 0.001 0.001"/>
+            </geometry>
+        </collision>
+    </link>
+    <!-- RIGHT WHEEL LINK -->
+    <joint name="right_wheel_joint" type="continuous">
+        <origin xyz="0.09 -0.0475 0.02" rpy="0 0 0"/>
+        <parent link="base_link"/>
+        <child link="right_wheel_1"/>
+        <axis xyz="-1.0 0.0 0.0"/>
+    </joint>
+    <link name="right_wheel_1">
+        <inertial>
+            <origin xyz="0.012500000000000108 0.0 -6.938893903907228e-18" rpy="0 0 0"/>
+            <mass value="0.6512177959195155"/>
+            <inertia ixx="0.000344" iyy="0.000206" izz="0.000206" ixy="0.0" iyz="0.0" ixz="0.0"/>
+        </inertial>
+        <visual>
+            <origin xyz="-0.09 0.0475 -0.02" rpy="0 0 0"/>
+            <geometry>
+                <mesh filename="file://$(find r2d10)/meshes/right_wheel_1.stl" scale="0.001 0.001 0.001"/>
+            </geometry>
+            <material name="black"/>
+        </visual>
+        <collision>
+            <origin xyz="-0.09 0.0475 -0.02" rpy="0 0 0"/>
+            <geometry>
+                <mesh filename="file://$(find r2d10)/meshes/right_wheel_1.stl" scale="0.001 0.001 0.001"/>
+            </geometry>
+        </collision>
+    </link>
+    <!-- ULTRASONIC FORWARD LINK -->
+    <joint name="ultrasonic_forward_joint" type="fixed">
+        <origin xyz="0.0 0.15 0.035" rpy="0 0 0"/>
+        <parent link="chassis"/>
+        <child link="ultrasonic_forward_1"/>
+    </joint>
+    <link name="ultrasonic_forward_1">
+        <inertial>
+            <origin xyz="-6.89984745874354e-13 0.005799256348663379 -6.55503359925369e-11" rpy="0 0 0"/>
+            <mass value="0.06306919012201337"/>
+            <inertia ixx="3e-06" iyy="1.2e-05" izz="1.2e-05" ixy="-0.0" iyz="0.0" ixz="-0.0"/>
+        </inertial>
+        <visual>
+            <origin xyz="-0.0 -0.15 -0.035" rpy="0 0 0"/>
+            <geometry>
+                <mesh filename="file://$(find r2d10)/meshes/ultrasonic_forward_1.stl" scale="0.001 0.001 0.001"/>
+            </geometry>
+            <material name="silver"/>
+        </visual>
+        <collision>
+            <origin xyz="-0.0 -0.15 -0.035" rpy="0 0 0"/>
+            <geometry>
+                <mesh filename="file://$(find r2d10)/meshes/ultrasonic_forward_1.stl" scale="0.001 0.001 0.001"/>
+            </geometry>
+        </collision>
+    </link>
+    <!-- ULTRASONIC LEFT LINK -->
+    <joint name="ultrasonic_left_joint" type="fixed">
+        <origin xyz="-0.15 0.0 0.035" rpy="0 0 0"/>
+        <parent link="chassis"/>
+        <child link="ultrasonic_left_1"/>
+    </joint>
+    <link name="ultrasonic_left_1">
+        <inertial>
+            <origin xyz="-0.005799256348663379 -6.899762237296075e-13 -6.55503359925369e-11" rpy="0 0 0"/>
+            <mass value="0.06306919012201337"/>
+            <inertia ixx="1.2e-05" iyy="3e-06" izz="1.2e-05" ixy="0.0" iyz="-0.0" ixz="-0.0"/>
+        </inertial>
+        <visual>
+            <origin xyz="0.15 -0.0 -0.035" rpy="0 0 0"/>
+            <geometry>
+                <mesh filename="file://$(find r2d10)/meshes/ultrasonic_left_1.stl" scale="0.001 0.001 0.001"/>
+            </geometry>
+            <material name="silver"/>
+        </visual>
+        <collision>
+            <origin xyz="0.15 -0.0 -0.035" rpy="0 0 0"/>
+            <geometry>
+                <mesh filename="file://$(find r2d10)/meshes/ultrasonic_left_1.stl" scale="0.001 0.001 0.001"/>
+            </geometry>
+        </collision>
+    </link>
+    <!-- ULTRASONIC RIGHT LINK -->
+    <joint name="ultrasonic_right_joint" type="fixed">
+        <origin xyz="0.15 0.0 0.035" rpy="0 0 0"/>
+        <parent link="chassis"/>
+        <child link="ultrasonic_right_1"/>
+    </joint>
+    <link name="ultrasonic_right_1">
+        <inertial>
+            <origin xyz="0.005799256348663379 6.899932680191004e-13 -6.55503359925369e-11" rpy="0 0 0"/>
+            <mass value="0.06306919012201337"/>
+            <inertia ixx="1.2e-05" iyy="3e-06" izz="1.2e-05" ixy="0.0" iyz="0.0" ixz="0.0"/>
+        </inertial>
+        <visual>
+            <origin xyz="-0.15 -0.0 -0.035" rpy="0 0 0"/>
+            <geometry>
+                <mesh filename="file://$(find r2d10)/meshes/ultrasonic_right_1.stl" scale="0.001 0.001 0.001"/>
+            </geometry>
+            <material name="silver"/>
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