Commit message: laser scan working, no map - need IMU integration to recieve map on rvis

File: install/r2d10/share/r2d10/urdf/assembly_3.urdf.xacro (robot description, xacro)
@@ -1,212 +1 @@
-<?xml version="1.0"?>
-<robot name="assembly_3" xmlns:xacro="http://www.ros.org/wiki/xacro">
-<!-- <xacro:include filename="$(find r2d10)/urdf/materials.xacro"/> -->
-<!-- <xacro:include filename="$(find-pkg-share r2d10)/urdf/assembly_3.trans"/>
-<xacro:include filename="$(find-pkg-share r2d10)/urdf/assembly_3.gazebo"/> -->
-<material name="silver"> <!-- colour is silver -->
-  <color rgba="0.700 0.700 0.700 1.000"/>
-</material>
-<material name="black"> <!-- wheels colour black -->
-  <color rgba="0 0 0 1"/>
-</material>
-<!-- physical part base_link -->
-<link name="base_link">
-  <inertial>   <!-- inertia link -->
-    <origin xyz="-6.745525765719935e-05 0.0012816498954868177 0.0354047315459432" rpy="0 0 0"/>  <!-- position & rotation -->
-    <mass value="37.821366170820795"/> <!-- mass (kg) -->
-    <inertia ixx="0.23125" iyy="0.223709" izz="0.423982" ixy="-0.000124" iyz="0.000747" ixz="-3.9e-05"/>  <!-- inertia matrix -->
-  </inertial>
-  <visual>
-    <origin xyz="0 0 0" rpy="0 0 0"/> <!-- position and rotation -->
-    <geometry>
-      <mesh filename="package://r2d10/meshes/base_link.stl" scale="0.001 0.001 0.001"/>
-    </geometry>
-    <material name="silver"/>
-  </visual>
-  <collision> <!-- physics collision shape -->
-    <origin xyz="0 0 0" rpy="0 0 0"/>
-    <geometry> <!-- shape of visual collision -->
-      <mesh filename="package://r2d10/meshes/base_link.stl" scale="0.001 0.001 0.001"/>
-    </geometry>
-  </collision>
-</link>
-<!-- link: physical part caster_1 -->
-<link name="caster_1">
-  <inertial>
-    <origin xyz="0.0 0.11 -0.0043996518255540636" rpy="0 0 0"/>
-    <mass value="0.0707011858312227"/>
-    <inertia ixx="6e-06" iyy="6e-06" izz="1e-05" ixy="0.0" iyz="-0.0" ixz="0.0"/>
-  </inertial>
-  <visual>
-    <origin xyz="-0.0 -0.0 -0.0" rpy="0 0 0"/>
-    <geometry>
-      <mesh filename="package://r2d10/meshes/caster_1.stl" scale="0.001 0.001 0.001"/>
-    </geometry>
-    <material name="silver"/>
-  </visual>
-  <collision>
-    <origin xyz="-0.0 -0.0 -0.0" rpy="0 0 0"/>
-    <geometry>
-      <mesh filename="package://r2d10/meshes/caster_1.stl" scale="0.001 0.001 0.001"/>
-    </geometry>
-  </collision>
-</link>
-<link name="left_wheel_1">
-  <inertial>
-    <origin xyz="-0.012500000000000011 0.0 0.0" rpy="0 0 0"/>
-    <mass value="0.6512177959195155"/>
-    <inertia ixx="0.000344" iyy="0.000206" izz="0.000206" ixy="0.0" iyz="-0.0" ixz="0.0"/>
-  </inertial>
-  <visual>
-    <origin xyz="0.085 0.0475 -0.02" rpy="0 0 0"/>
-    <geometry>
-      <mesh filename="package://r2d10/meshes/left_wheel_1.stl" scale="0.001 0.001 0.001"/>
-    </geometry>
-    <material name="black"/>
-  </visual>
-  <collision>
-    <origin xyz="0.085 0.0475 -0.02" rpy="0 0 0"/>
-    <geometry>
-      <mesh filename="package://r2d10/meshes/left_wheel_1.stl" scale="0.001 0.001 0.001"/>
-    </geometry>
-  </collision>
-</link>
-<link name="right_wheel_1">
-  <inertial>
-    <origin xyz="0.012500000000000108 0.0 -6.938893903907228e-18" rpy="0 0 0"/>
-    <mass value="0.6512177959195155"/>
-    <inertia ixx="0.000344" iyy="0.000206" izz="0.000206" ixy="0.0" iyz="0.0" ixz="0.0"/>
-  </inertial>
-  <visual>
-    <origin xyz="-0.09 0.0475 -0.02" rpy="0 0 0"/>
-    <geometry>
-      <mesh filename="package://r2d10/meshes/right_wheel_1.stl" scale="0.001 0.001 0.001"/>
-    </geometry>
-    <material name="black"/>
-  </visual>
-  <collision>
-    <origin xyz="-0.09 0.0475 -0.02" rpy="0 0 0"/>
-    <geometry>
-      <mesh filename="package://r2d10/meshes/right_wheel_1.stl" scale="0.001 0.001 0.001"/>
-    </geometry>
-  </collision>
-</link>
-<link name="ultrasonic_forward_1">
-  <inertial>
-    <origin xyz="-6.89984745874354e-13 0.005799256348663379 -6.55503359925369e-11" rpy="0 0 0"/>
-    <mass value="0.06306919012201337"/>
-    <inertia ixx="3e-06" iyy="1.2e-05" izz="1.2e-05" ixy="-0.0" iyz="0.0" ixz="-0.0"/>
-  </inertial>
-  <visual>
-    <origin xyz="-0.0 -0.15 -0.035" rpy="0 0 0"/>
-    <geometry>
-      <mesh filename="package://r2d10/meshes/ultrasonic_forward_1.stl" scale="0.001 0.001 0.001"/>
-    </geometry>
-    <material name="silver"/>
-  </visual>
-  <collision>
-    <origin xyz="-0.0 -0.15 -0.035" rpy="0 0 0"/>
-    <geometry>
-      <mesh filename="package://r2d10/meshes/ultrasonic_forward_1.stl" scale="0.001 0.001 0.001"/>
-    </geometry>
-  </collision>
-</link>
-<link name="ultrasonic_left_1">
-  <inertial>
-    <origin xyz="-0.005799256348663379 -6.899762237296075e-13 -6.55503359925369e-11" rpy="0 0 0"/>
-    <mass value="0.06306919012201337"/>
-    <inertia ixx="1.2e-05" iyy="3e-06" izz="1.2e-05" ixy="0.0" iyz="-0.0" ixz="-0.0"/>
-  </inertial>
-  <visual>
-    <origin xyz="0.15 -0.0 -0.035" rpy="0 0 0"/>
-    <geometry>
-      <mesh filename="package://r2d10/meshes/ultrasonic_left_1.stl" scale="0.001 0.001 0.001"/>
-    </geometry>
-    <material name="silver"/>
-  </visual>
-  <collision>
-    <origin xyz="0.15 -0.0 -0.035" rpy="0 0 0"/>
-    <geometry>
-      <mesh filename="package://r2d10/meshes/ultrasonic_left_1.stl" scale="0.001 0.001 0.001"/>
-    </geometry>
-  </collision>
-</link>
-<link name="ultrasonic_right_1">
-  <inertial>
-    <origin xyz="0.005799256348663379 6.899932680191004e-13 -6.55503359925369e-11" rpy="0 0 0"/>
-    <mass value="0.06306919012201337"/>
-    <inertia ixx="1.2e-05" iyy="3e-06" izz="1.2e-05" ixy="0.0" iyz="0.0" ixz="0.0"/>
-  </inertial>
-  <visual>
-    <origin xyz="-0.15 -0.0 -0.035" rpy="0 0 0"/>
-    <geometry>
-      <mesh filename="package://r2d10/meshes/ultrasonic_right_1.stl" scale="0.001 0.001 0.001"/>
-    </geometry>
-    <material name="silver"/>
-  </visual>
-  <collision>
-    <origin xyz="-0.15 -0.0 -0.035" rpy="0 0 0"/>
-    <geometry>
-      <mesh filename="package://r2d10/meshes/ultrasonic_right_1.stl" scale="0.001 0.001 0.001"/>
-    </geometry>
-  </collision>
-</link>
-<link name="lidar_1">
-  <inertial>
-    <origin xyz="7.385233546074017e-18 0.0 0.01999999999999999" rpy="0 0 0"/>
-    <mass value="1.2084136142033137"/>
-    <inertia ixx="0.000531" iyy="0.000531" izz="0.00074" ixy="0.0" iyz="0.0" ixz="0.0"/>
-  </inertial>
-  <visual>
-    <origin xyz="-0.0 -0.0 -0.07" rpy="0 0 0"/>
-    <geometry>
-      <mesh filename="package://r2d10/meshes/lidar_1.stl" scale="0.001 0.001 0.001"/>
-    </geometry>
-    <material name="silver"/>
-  </visual>
-  <collision>
-    <origin xyz="-0.0 -0.0 -0.07" rpy="0 0 0"/>
-    <geometry>
-      <mesh filename="package://r2d10/meshes/lidar_1.stl" scale="0.001 0.001 0.001"/>
-    </geometry>
-  </collision>
-</link>
-<!-- joint part connectors such as type and name -->
-<joint name="Rigid 1" type="fixed">
-  <origin xyz="0.0 0.0 0.0" rpy="0 0 0"/>
-  <parent link="base_link"/>
-  <child link="caster_1"/>
-</joint>
-<joint name="Revolute 2" type="continuous">
-  <origin xyz="-0.085 -0.0475 0.02" rpy="0 0 0"/>
-  <parent link="base_link"/>
-  <child link="left_wheel_1"/>
-  <axis xyz="-1.0 0.0 0.0"/>
-</joint>
-<joint name="Revolute 3" type="continuous">
-  <origin xyz="0.09 -0.0475 0.02" rpy="0 0 0"/>
-  <parent link="base_link"/>
-  <child link="right_wheel_1"/>
-  <axis xyz="1.0 0.0 0.0"/>
-</joint>
-<joint name="Rigid 5" type="fixed">
-  <origin xyz="0.0 0.15 0.035" rpy="0 0 0"/>
-  <parent link="base_link"/>
-  <child link="ultrasonic_forward_1"/>
-</joint>
-<joint name="Rigid 6" type="fixed">
-  <origin xyz="-0.15 0.0 0.035" rpy="0 0 0"/>
-  <parent link="base_link"/>
-  <child link="ultrasonic_left_1"/>
-</joint>
-<joint name="Rigid 7" type="fixed">
-  <origin xyz="0.15 0.0 0.035" rpy="0 0 0"/>
-  <parent link="base_link"/>
-  <child link="ultrasonic_right_1"/>
-</joint>
-<joint name="Rigid 9" type="fixed">
-  <origin xyz="0.0 0.0 0.07" rpy="0 0 0"/>
-  <parent link="base_link"/>
-  <child link="lidar_1"/>
-</joint>
-</robot>
+/home/group10/ros2_ws/src/r2d10/urdf/assembly_3.urdf.xacro

File: install/r2d10/share/r2d10/urdf/materials.xacro (robot description, xacro)
@@ -1,6 +1 @@
-<?xml version="1.0" ?>
-<robot name="assembly_3" xmlns:xacro="http://www.ros.org/wiki/xacro" >
-<material name="silver">
-  <color rgba="0.700 0.700 0.700 1.000"/>
-</material>
-</robot>
+/home/group10/ros2_ws/src/r2d10/urdf/materials.xacro

Commit message: try running all terminals and check if map being recieved on RVIS - debug if not

File: install/r2d10/share/r2d10/urdf/assembly_3.urdf.xacro (robot description, xacro)
@@ -1 +1,212 @@
-/home/group10/ros2_ws/src/r2d10/urdf/assembly_3.urdf.xacro
+<?xml version="1.0"?>
+<robot name="assembly_3" xmlns:xacro="http://www.ros.org/wiki/xacro">
+<!-- <xacro:include filename="$(find r2d10)/urdf/materials.xacro"/> -->
+<!-- <xacro:include filename="$(find-pkg-share r2d10)/urdf/assembly_3.trans"/>
+<xacro:include filename="$(find-pkg-share r2d10)/urdf/assembly_3.gazebo"/> -->
+<material name="silver"> <!-- colour is silver -->
+  <color rgba="0.700 0.700 0.700 1.000"/>
+</material>
+<material name="black"> <!-- wheels colour black -->
+  <color rgba="0 0 0 1"/>
+</material>
+<!-- physical part base_link -->
+<link name="base_link">
+  <inertial>   <!-- inertia link -->
+    <origin xyz="-6.745525765719935e-05 0.0012816498954868177 0.0354047315459432" rpy="0 0 0"/>  <!-- position & rotation -->
+    <mass value="37.821366170820795"/> <!-- mass (kg) -->
+    <inertia ixx="0.23125" iyy="0.223709" izz="0.423982" ixy="-0.000124" iyz="0.000747" ixz="-3.9e-05"/>  <!-- inertia matrix -->
+  </inertial>
+  <visual>
+    <origin xyz="0 0 0" rpy="0 0 0"/> <!-- position and rotation -->
+    <geometry>
+      <mesh filename="package://r2d10/meshes/base_link.stl" scale="0.001 0.001 0.001"/>
+    </geometry>
+    <material name="silver"/>
+  </visual>
+  <collision> <!-- physics collision shape -->
+    <origin xyz="0 0 0" rpy="0 0 0"/>
+    <geometry> <!-- shape of visual collision -->
+      <mesh filename="package://r2d10/meshes/base_link.stl" scale="0.001 0.001 0.001"/>
+    </geometry>
+  </collision>
+</link>
+<!-- link: physical part caster_1 -->
+<link name="caster_1">
+  <inertial>
+    <origin xyz="0.0 0.11 -0.0043996518255540636" rpy="0 0 0"/>
+    <mass value="0.0707011858312227"/>
+    <inertia ixx="6e-06" iyy="6e-06" izz="1e-05" ixy="0.0" iyz="-0.0" ixz="0.0"/>
+  </inertial>
+  <visual>
+    <origin xyz="-0.0 -0.0 -0.0" rpy="0 0 0"/>
+    <geometry>
+      <mesh filename="package://r2d10/meshes/caster_1.stl" scale="0.001 0.001 0.001"/>
+    </geometry>
+    <material name="silver"/>
+  </visual>
+  <collision>
+    <origin xyz="-0.0 -0.0 -0.0" rpy="0 0 0"/>
+    <geometry>
+      <mesh filename="package://r2d10/meshes/caster_1.stl" scale="0.001 0.001 0.001"/>
+    </geometry>
+  </collision>
+</link>
+<link name="left_wheel_1">
+  <inertial>
+    <origin xyz="-0.012500000000000011 0.0 0.0" rpy="0 0 0"/>
+    <mass value="0.6512177959195155"/>
+    <inertia ixx="0.000344" iyy="0.000206" izz="0.000206" ixy="0.0" iyz="-0.0" ixz="0.0"/>
+  </inertial>
+  <visual>
+    <origin xyz="0.085 0.0475 -0.02" rpy="0 0 0"/>
+    <geometry>
+      <mesh filename="package://r2d10/meshes/left_wheel_1.stl" scale="0.001 0.001 0.001"/>
+    </geometry>
+    <material name="black"/>
+  </visual>
+  <collision>
+    <origin xyz="0.085 0.0475 -0.02" rpy="0 0 0"/>
+    <geometry>
+      <mesh filename="package://r2d10/meshes/left_wheel_1.stl" scale="0.001 0.001 0.001"/>
+    </geometry>
+  </collision>
+</link>
+<link name="right_wheel_1">
+  <inertial>
+    <origin xyz="0.012500000000000108 0.0 -6.938893903907228e-18" rpy="0 0 0"/>
+    <mass value="0.6512177959195155"/>
+    <inertia ixx="0.000344" iyy="0.000206" izz="0.000206" ixy="0.0" iyz="0.0" ixz="0.0"/>
+  </inertial>
+  <visual>
+    <origin xyz="-0.09 0.0475 -0.02" rpy="0 0 0"/>
+    <geometry>
+      <mesh filename="package://r2d10/meshes/right_wheel_1.stl" scale="0.001 0.001 0.001"/>
+    </geometry>
+    <material name="black"/>
+  </visual>
+  <collision>
+    <origin xyz="-0.09 0.0475 -0.02" rpy="0 0 0"/>
+    <geometry>
+      <mesh filename="package://r2d10/meshes/right_wheel_1.stl" scale="0.001 0.001 0.001"/>
+    </geometry>
+  </collision>
+</link>
+<link name="ultrasonic_forward_1">
+  <inertial>
+    <origin xyz="-6.89984745874354e-13 0.005799256348663379 -6.55503359925369e-11" rpy="0 0 0"/>
+    <mass value="0.06306919012201337"/>
+    <inertia ixx="3e-06" iyy="1.2e-05" izz="1.2e-05" ixy="-0.0" iyz="0.0" ixz="-0.0"/>
+  </inertial>
+  <visual>
+    <origin xyz="-0.0 -0.15 -0.035" rpy="0 0 0"/>
+    <geometry>
+      <mesh filename="package://r2d10/meshes/ultrasonic_forward_1.stl" scale="0.001 0.001 0.001"/>
+    </geometry>
+    <material name="silver"/>
+  </visual>
+  <collision>
+    <origin xyz="-0.0 -0.15 -0.035" rpy="0 0 0"/>
+    <geometry>
+      <mesh filename="package://r2d10/meshes/ultrasonic_forward_1.stl" scale="0.001 0.001 0.001"/>
+    </geometry>
+  </collision>
+</link>
+<link name="ultrasonic_left_1">
+  <inertial>
+    <origin xyz="-0.005799256348663379 -6.899762237296075e-13 -6.55503359925369e-11" rpy="0 0 0"/>
+    <mass value="0.06306919012201337"/>
+    <inertia ixx="1.2e-05" iyy="3e-06" izz="1.2e-05" ixy="0.0" iyz="-0.0" ixz="-0.0"/>
+  </inertial>
+  <visual>
+    <origin xyz="0.15 -0.0 -0.035" rpy="0 0 0"/>
+    <geometry>
+      <mesh filename="package://r2d10/meshes/ultrasonic_left_1.stl" scale="0.001 0.001 0.001"/>
+    </geometry>
+    <material name="silver"/>
+  </visual>
+  <collision>
+    <origin xyz="0.15 -0.0 -0.035" rpy="0 0 0"/>
+    <geometry>
+      <mesh filename="package://r2d10/meshes/ultrasonic_left_1.stl" scale="0.001 0.001 0.001"/>
+    </geometry>
+  </collision>
+</link>
+<link name="ultrasonic_right_1">
+  <inertial>
+    <origin xyz="0.005799256348663379 6.899932680191004e-13 -6.55503359925369e-11" rpy="0 0 0"/>
+    <mass value="0.06306919012201337"/>
+    <inertia ixx="1.2e-05" iyy="3e-06" izz="1.2e-05" ixy="0.0" iyz="0.0" ixz="0.0"/>
+  </inertial>
+  <visual>
+    <origin xyz="-0.15 -0.0 -0.035" rpy="0 0 0"/>
+    <geometry>
+      <mesh filename="package://r2d10/meshes/ultrasonic_right_1.stl" scale="0.001 0.001 0.001"/>
+    </geometry>
+    <material name="silver"/>
+  </visual>
+  <collision>
+    <origin xyz="-0.15 -0.0 -0.035" rpy="0 0 0"/>
+    <geometry>
+      <mesh filename="package://r2d10/meshes/ultrasonic_right_1.stl" scale="0.001 0.001 0.001"/>
+    </geometry>
+  </collision>
+</link>
+<link name="lidar_1">
+  <inertial>
+    <origin xyz="7.385233546074017e-18 0.0 0.01999999999999999" rpy="0 0 0"/>
+    <mass value="1.2084136142033137"/>
+    <inertia ixx="0.000531" iyy="0.000531" izz="0.00074" ixy="0.0" iyz="0.0" ixz="0.0"/>
+  </inertial>
+  <visual>
+    <origin xyz="-0.0 -0.0 -0.07" rpy="0 0 0"/>
+    <geometry>
+      <mesh filename="package://r2d10/meshes/lidar_1.stl" scale="0.001 0.001 0.001"/>
+    </geometry>
+    <material name="silver"/>
+  </visual>
+  <collision>
+    <origin xyz="-0.0 -0.0 -0.07" rpy="0 0 0"/>
+    <geometry>
+      <mesh filename="package://r2d10/meshes/lidar_1.stl" scale="0.001 0.001 0.001"/>
+    </geometry>
+  </collision>
+</link>
+<!-- joint part connectors such as type and name -->
+<joint name="Rigid 1" type="fixed">
+  <origin xyz="0.0 0.0 0.0" rpy="0 0 0"/>
+  <parent link="base_link"/>
+  <child link="caster_1"/>
+</joint>
+<joint name="Revolute 2" type="continuous">
+  <origin xyz="-0.085 -0.0475 0.02" rpy="0 0 0"/>
+  <parent link="base_link"/>
+  <child link="left_wheel_1"/>
+  <axis xyz="-1.0 0.0 0.0"/>
+</joint>
+<joint name="Revolute 3" type="continuous">
+  <origin xyz="0.09 -0.0475 0.02" rpy="0 0 0"/>
+  <parent link="base_link"/>
+  <child link="right_wheel_1"/>
+  <axis xyz="1.0 0.0 0.0"/>
+</joint>
+<joint name="Rigid 5" type="fixed">
+  <origin xyz="0.0 0.15 0.035" rpy="0 0 0"/>
+  <parent link="base_link"/>
+  <child link="ultrasonic_forward_1"/>
+</joint>
+<joint name="Rigid 6" type="fixed">
+  <origin xyz="-0.15 0.0 0.035" rpy="0 0 0"/>
+  <parent link="base_link"/>
+  <child link="ultrasonic_left_1"/>
+</joint>
+<joint name="Rigid 7" type="fixed">
+  <origin xyz="0.15 0.0 0.035" rpy="0 0 0"/>
+  <parent link="base_link"/>
+  <child link="ultrasonic_right_1"/>
+</joint>
+<joint name="Rigid 9" type="fixed">
+  <origin xyz="0.0 0.0 0.07" rpy="0 0 0"/>
+  <parent link="base_link"/>
+  <child link="lidar_1"/>
+</joint>
+</robot>

File: install/r2d10/share/r2d10/urdf/materials.xacro (robot description, xacro)
@@ -1 +1,6 @@
-/home/group10/ros2_ws/src/r2d10/urdf/materials.xacro
+<?xml version="1.0" ?>
+<robot name="assembly_3" xmlns:xacro="http://www.ros.org/wiki/xacro" >
+<material name="silver">
+  <color rgba="0.700 0.700 0.700 1.000"/>
+</material>
+</robot>

Commit message: SLAM working! - create 2 maps, add nav, face detection

File: install/r2d10/share/r2d10/urdf/assembly_3.urdf.xacro (robot description, xacro)
@@ -68,5 +68,5 @@
     <joint name="left_wheel_joint" type="continuous">
         <origin xyz="-0.085 -0.0475 0.02" rpy="0 0 0"/>
-        <parent link="base_link"/>
+        <parent link="chassis"/>
         <child link="left_wheel_1"/>
         <axis xyz="-1.0 0.0 0.0"/>
@@ -95,5 +95,5 @@
     <joint name="right_wheel_joint" type="continuous">
         <origin xyz="0.09 -0.0475 0.02" rpy="0 0 0"/>
-        <parent link="base_link"/>
+        <parent link="chassis"/>
         <child link="right_wheel_1"/>
         <axis xyz="-1.0 0.0 0.0"/>
@@ -226,5 +226,5 @@
     <joint name="imu_joint" type="fixed">
         <origin xyz="0 0 0" rpy="0 0 0" />
-        <parent link="base_link"/>
+        <parent link="chassis"/>
         <child link="imu_link" />
     </joint>

Commit message: working slam, map created, nav stack begun, face detection integration started

File: install/r2d10/share/r2d10/urdf/assembly_3.urdf.xacro (robot description, xacro)
@@ -17,5 +17,5 @@
         <parent link="base_link"/>
         <child link="chassis"/>
-        <origin xyz="0 0 0" rpy="0 0 0"/>
+        <origin xyz="0 0 0" rpy="0 0 -1.5708"/>
     </joint>
     <link name="chassis">
@@ -247,3 +247,49 @@
         <mu2>1.0</mu2>
     </gazebo>
+    <!-- CAMERA LINK -->
+    <!-- <link name="camera_link">
+    <inertial>
+      <origin xyz="0 0 0" rpy="0 0 0"/>
+      <mass value="0.1"/>
+      <inertia ixx="1e-4" iyy="1e-4" izz="1e-4" ixy="0" iyz="0" ixz="0"/>
+    </inertial>
+    <visual>
+      <origin xyz="0 0 0" rpy="0 0 0"/>
+      <geometry>
+        <box size="0.05 0.05 0.05"/>
+      </geometry>
+      <material name="black"/>
+    </visual>
+    <collision>
+      <origin xyz="0 0 0" rpy="0 0 0"/>
+      <geometry>
+        <box size="0.05 0.05 0.05"/>
+      </geometry>
+    </collision>
+  </link> -->
+    <!-- <gazebo reference="camera_link">
+    <sensor name="front_camera" type="camera">
+      <always_on>1</always_on>
+      <update_rate>10</update_rate>
+      <visualize>true</visualize>
+      <topic>/camera/image_raw</topic>
+      <camera>
+        <horizontal_fov>1.047</horizontal_fov>
+        <image>
+          <width>640</width>
+          <height>480</height>
+          <format>R8G8B8</format>
+        </image>
+        <clip>
+          <near>0.1</near>
+          <far>20.0</far>
+        </clip>
+      </camera>
+    </sensor> -->
+  <!-- <joint name="camera_mount" type="fixed">
+    <parent link="base_link"/>
+    <child link="camera_link"/>
+    <origin xyz="0 0 0.12" rpy="0 0 0"/>
+  </joint> -->
+  <!-- </gazebo> -->
 </robot>
