Commit message: face detection node working, camera needs to be added

File: install/r2d10/share/r2d10/urdf/assembly_3.urdf.xacro (robot description, xacro)
@@ -1,295 +1 @@
-<?xml version="1.0"?>
-<robot name="assembly_3" xmlns:xacro="http://www.ros.org/wiki/xacro">
-    <xacro:include filename="$(find r2d10)/urdf/r2d10.gazebo" />
-    <xacro:include filename="$(find r2d10)/urdf/inertial_macros.xacro" />
-    <!-- MATERIALS -->
-    <material name="silver">
-        <color rgba="0.700 0.700 0.700 1.000"/>
-    </material>
-    <material name="black">
-        <color rgba="0 0 0 1"/>
-    </material>
-    <!-- BASE LINK -->
-    <link name="base_link">
-    </link>
-    <!-- CHASSIS (your base_link visual/collision) -->
-    <joint name="chassis_joint" type="fixed">
-        <parent link="base_link"/>
-        <child link="chassis"/>
-        <origin xyz="0 0 0" rpy="0 0 -1.5708"/>
-    </joint>
-    <link name="chassis">
-        <inertial>
-            <origin xyz="-6.745525765719935e-05 0.0012816498954868177 0.0354047315459432" rpy="0 0 0"/>
-            <mass value="37.821366170820795"/>
-            <inertia ixx="0.23125" iyy="0.223709" izz="0.423982" ixy="-0.000124" iyz="0.000747" ixz="-3.9e-05"/>
-        </inertial>
-        <visual>
-            <origin xyz="0 0 0" rpy="0 0 0"/>
-            <geometry>
-                <mesh filename="file://$(find r2d10)/meshes/base_link.stl" scale="0.001 0.001 0.001"/>
-            </geometry>
-            <material name="silver"/>
-        </visual>
-        <collision>
-            <origin xyz="0 0 0" rpy="0 0 0"/>
-            <geometry>
-                <mesh filename="file://$(find r2d10)/meshes/base_link.stl" scale="0.001 0.001 0.001"/>
-            </geometry>
-        </collision>
-    </link>
-    <!-- CASTER LINK -->
-    <joint name="caster_joint" type="fixed">
-        <origin xyz="0.0 0.0 0.0" rpy="0 0 0"/>
-        <parent link="chassis"/>
-        <child link="caster_1"/>
-    </joint>
-    <link name="caster_1">
-        <inertial>
-            <origin xyz="0.0 0.11 -0.0043996518255540636" rpy="0 0 0"/>
-            <mass value="0.0707011858312227"/>
-            <inertia ixx="6e-06" iyy="6e-06" izz="1e-05" ixy="0.0" iyz="-0.0" ixz="0.0"/>
-        </inertial>
-        <visual>
-            <origin xyz="-0.0 -0.0 -0.0" rpy="0 0 0"/>
-            <geometry>
-                <mesh filename="file://$(find r2d10)/meshes/caster_1.stl" scale="0.001 0.001 0.001"/>
-            </geometry>
-            <material name="silver"/>
-        </visual>
-        <collision>
-            <origin xyz="-0.0 -0.0 -0.0" rpy="0 0 0"/>
-            <geometry>
-                <mesh filename="file://$(find r2d10)/meshes/caster_1.stl" scale="0.001 0.001 0.001"/>
-            </geometry>
-        </collision>
-    </link>
-    <!-- LEFT WHEEL LINK -->
-    <joint name="left_wheel_joint" type="continuous">
-        <origin xyz="-0.085 -0.0475 0.02" rpy="0 0 0"/>
-        <parent link="chassis"/>
-        <child link="left_wheel_1"/>
-        <axis xyz="-1.0 0.0 0.0"/>
-    </joint>
-    <link name="left_wheel_1">
-        <inertial>
-            <origin xyz="-0.012500000000000011 0.0 0.0" rpy="0 0 0"/>
-            <mass value="0.6512177959195155"/>
-            <inertia ixx="0.000344" iyy="0.000206" izz="0.000206" ixy="0.0" iyz="-0.0" ixz="0.0"/>
-        </inertial>
-        <visual>
-            <origin xyz="0.085 0.0475 -0.02" rpy="0 0 0"/>
-            <geometry>
-                <mesh filename="file://$(find r2d10)/meshes/left_wheel_1.stl" scale="0.001 0.001 0.001"/>
-            </geometry>
-            <material name="black"/>
-        </visual>
-        <collision>
-            <origin xyz="0.085 0.0475 -0.02" rpy="0 0 0"/>
-            <geometry>
-               <mesh filename="file://$(find r2d10)/meshes/left_wheel_1.stl" scale="0.001 0.001 0.001"/>
-            </geometry>
-        </collision>
-    </link>
-    <!-- RIGHT WHEEL LINK -->
-    <joint name="right_wheel_joint" type="continuous">
-        <origin xyz="0.09 -0.0475 0.02" rpy="0 0 0"/>
-        <parent link="chassis"/>
-        <child link="right_wheel_1"/>
-        <axis xyz="-1.0 0.0 0.0"/>
-    </joint>
-    <link name="right_wheel_1">
-        <inertial>
-            <origin xyz="0.012500000000000108 0.0 -6.938893903907228e-18" rpy="0 0 0"/>
-            <mass value="0.6512177959195155"/>
-            <inertia ixx="0.000344" iyy="0.000206" izz="0.000206" ixy="0.0" iyz="0.0" ixz="0.0"/>
-        </inertial>
-        <visual>
-            <origin xyz="-0.09 0.0475 -0.02" rpy="0 0 0"/>
-            <geometry>
-                <mesh filename="file://$(find r2d10)/meshes/right_wheel_1.stl" scale="0.001 0.001 0.001"/>
-            </geometry>
-            <material name="black"/>
-        </visual>
-        <collision>
-            <origin xyz="-0.09 0.0475 -0.02" rpy="0 0 0"/>
-            <geometry>
-                <mesh filename="file://$(find r2d10)/meshes/right_wheel_1.stl" scale="0.001 0.001 0.001"/>
-            </geometry>
-        </collision>
-    </link>
-    <!-- ULTRASONIC FORWARD LINK -->
-    <joint name="ultrasonic_forward_joint" type="fixed">
-        <origin xyz="0.0 0.15 0.035" rpy="0 0 0"/>
-        <parent link="chassis"/>
-        <child link="ultrasonic_forward_1"/>
-    </joint>
-    <link name="ultrasonic_forward_1">
-        <inertial>
-            <origin xyz="-6.89984745874354e-13 0.005799256348663379 -6.55503359925369e-11" rpy="0 0 0"/>
-            <mass value="0.06306919012201337"/>
-            <inertia ixx="3e-06" iyy="1.2e-05" izz="1.2e-05" ixy="-0.0" iyz="0.0" ixz="-0.0"/>
-        </inertial>
-        <visual>
-            <origin xyz="-0.0 -0.15 -0.035" rpy="0 0 0"/>
-            <geometry>
-                <mesh filename="file://$(find r2d10)/meshes/ultrasonic_forward_1.stl" scale="0.001 0.001 0.001"/>
-            </geometry>
-            <material name="silver"/>
-        </visual>
-        <collision>
-            <origin xyz="-0.0 -0.15 -0.035" rpy="0 0 0"/>
-            <geometry>
-                <mesh filename="file://$(find r2d10)/meshes/ultrasonic_forward_1.stl" scale="0.001 0.001 0.001"/>
-            </geometry>
-        </collision>
-    </link>
-    <!-- ULTRASONIC LEFT LINK -->
-    <joint name="ultrasonic_left_joint" type="fixed">
-        <origin xyz="-0.15 0.0 0.035" rpy="0 0 0"/>
-        <parent link="chassis"/>
-        <child link="ultrasonic_left_1"/>
-    </joint>
-    <link name="ultrasonic_left_1">
-        <inertial>
-            <origin xyz="-0.005799256348663379 -6.899762237296075e-13 -6.55503359925369e-11" rpy="0 0 0"/>
-            <mass value="0.06306919012201337"/>
-            <inertia ixx="1.2e-05" iyy="3e-06" izz="1.2e-05" ixy="0.0" iyz="-0.0" ixz="-0.0"/>
-        </inertial>
-        <visual>
-            <origin xyz="0.15 -0.0 -0.035" rpy="0 0 0"/>
-            <geometry>
-                <mesh filename="file://$(find r2d10)/meshes/ultrasonic_left_1.stl" scale="0.001 0.001 0.001"/>
-            </geometry>
-            <material name="silver"/>
-        </visual>
-        <collision>
-            <origin xyz="0.15 -0.0 -0.035" rpy="0 0 0"/>
-            <geometry>
-                <mesh filename="file://$(find r2d10)/meshes/ultrasonic_left_1.stl" scale="0.001 0.001 0.001"/>
-            </geometry>
-        </collision>
-    </link>
-    <!-- ULTRASONIC RIGHT LINK -->
-    <joint name="ultrasonic_right_joint" type="fixed">
-        <origin xyz="0.15 0.0 0.035" rpy="0 0 0"/>
-        <parent link="chassis"/>
-        <child link="ultrasonic_right_1"/>
-    </joint>
-    <link name="ultrasonic_right_1">
-        <inertial>
-            <origin xyz="0.005799256348663379 6.899932680191004e-13 -6.55503359925369e-11" rpy="0 0 0"/>
-            <mass value="0.06306919012201337"/>
-            <inertia ixx="1.2e-05" iyy="3e-06" izz="1.2e-05" ixy="0.0" iyz="0.0" ixz="0.0"/>
-        </inertial>
-        <visual>
-            <origin xyz="-0.15 -0.0 -0.035" rpy="0 0 0"/>
-            <geometry>
-                <mesh filename="file://$(find r2d10)/meshes/ultrasonic_right_1.stl" scale="0.001 0.001 0.001"/>
-            </geometry>
-            <material name="silver"/>
-        </visual>
-        <collision>
-            <origin xyz="-0.15 -0.0 -0.035" rpy="0 0 0"/>
-            <geometry>
-                <mesh filename="file://$(find r2d10)/meshes/ultrasonic_right_1.stl" scale="0.001 0.001 0.001"/>
-            </geometry>
-        </collision>
-    </link>
-    <!-- LIDAR LINK -->
-    <joint name="lidar_joint" type="fixed">
-        <origin xyz="0.0 0.0 0.07" rpy="0 0 0"/>
-        <parent link="chassis"/>
-        <child link="lidar_1"/>
-    </joint>
-    <link name="lidar_1">
-        <inertial>
-            <origin xyz="7.385233546074017e-18 0.0 0.01999999999999999" rpy="0 0 0"/>
-            <mass value="1.2084136142033137"/>
-            <inertia ixx="0.000531" iyy="0.000531" izz="0.00074" ixy="0.0" iyz="0.0" ixz="0.0"/>
-        </inertial>
-        <visual>
-            <origin xyz="-0.0 -0.0 -0.07" rpy="0 0 0"/>
-            <geometry>
-                <mesh filename="file://$(find r2d10)/meshes/lidar_1.stl" scale="0.001 0.001 0.001"/>
-            </geometry>
-            <material name="silver"/>
-        </visual>
-        <collision>
-            <origin xyz="-0.0 -0.0 -0.07" rpy="0 0 0"/>
-            <geometry>
-                <mesh filename="file://$(find r2d10)/meshes/lidar_1.stl" scale="0.001 0.001 0.001"/>
-            </geometry>
-        </collision>
-    </link>
-    <!-- IMU SENSOR LINK -->
-    <joint name="imu_joint" type="fixed">
-        <origin xyz="0 0 0" rpy="0 0 0" />
-        <parent link="chassis"/>
-        <child link="imu_link" />
-    </joint>
-    <link name="imu_link" />
-    <!-- GAZEBO FRICTION PARAMETERS -->
-    <gazebo reference="left_wheel_1">
-        <mu1>1.0</mu1>
-        <mu2>1.0</mu2>
-    </gazebo>
-    <gazebo reference="right_wheel_1">
-        <mu1>1.0</mu1>
-        <mu2>1.0</mu2>
-    </gazebo>
-    <gazebo reference="caster_1">
-        <mu1>0.000001</mu1>
-        <mu2>0.000001</mu2>
-    </gazebo>
-    <gazebo reference="base_link">
-        <mu1>1.0</mu1>
-        <mu2>1.0</mu2>
-    </gazebo>
-    <!-- CAMERA LINK -->
-    <!-- <link name="camera_link">
-    <inertial>
-      <origin xyz="0 0 0" rpy="0 0 0"/>
-      <mass value="0.1"/>
-      <inertia ixx="1e-4" iyy="1e-4" izz="1e-4" ixy="0" iyz="0" ixz="0"/>
-    </inertial>
-    <visual>
-      <origin xyz="0 0 0" rpy="0 0 0"/>
-      <geometry>
-        <box size="0.05 0.05 0.05"/>
-      </geometry>
-      <material name="black"/>
-    </visual>
-    <collision>
-      <origin xyz="0 0 0" rpy="0 0 0"/>
-      <geometry>
-        <box size="0.05 0.05 0.05"/>
-      </geometry>
-    </collision>
-  </link> -->
-    <!-- <gazebo reference="camera_link">
-    <sensor name="front_camera" type="camera">
-      <always_on>1</always_on>
-      <update_rate>10</update_rate>
-      <visualize>true</visualize>
-      <topic>/camera/image_raw</topic>
-      <camera>
-        <horizontal_fov>1.047</horizontal_fov>
-        <image>
-          <width>640</width>
-          <height>480</height>
-          <format>R8G8B8</format>
-        </image>
-        <clip>
-          <near>0.1</near>
-          <far>20.0</far>
-        </clip>
-      </camera>
-    </sensor> -->
-  <!-- <joint name="camera_mount" type="fixed">
-    <parent link="base_link"/>
-    <child link="camera_link"/>
-    <origin xyz="0 0 0.12" rpy="0 0 0"/>
-  </joint> -->
-  <!-- </gazebo> -->
-</robot>
+/home/group10/ros2_ws/src/r2d10/urdf/assembly_3.urdf.xacro

File: src/r2d10/urdf/assembly_3.urdf.xacro (robot description, xacro)
@@ -248,5 +248,5 @@
     </gazebo>
     <!-- CAMERA LINK -->
-    <!-- <link name="camera_link">
+    <link name="camera_link">
     <inertial>
       <origin xyz="0 0 0" rpy="0 0 0"/>
@@ -267,6 +267,11 @@
       </geometry>
     </collision>
-  </link> -->
-    <!-- <gazebo reference="camera_link">
+  </link>
+<joint name="camera_mount" type="fixed">
+    <parent link="chassis"/>
+    <child link="camera_link"/>
+    <origin xyz="0 0 0.12" rpy="0 0 0"/>
+  </joint>
+    <gazebo reference="camera_link">
     <sensor name="front_camera" type="camera">
       <always_on>1</always_on>
@@ -286,10 +291,5 @@
         </clip>
       </camera>
-    </sensor> -->
-  <!-- <joint name="camera_mount" type="fixed">
-    <parent link="base_link"/>
-    <child link="camera_link"/>
-    <origin xyz="0 0 0.12" rpy="0 0 0"/>
-  </joint> -->
-  <!-- </gazebo> -->
+    </sensor>
+  </gazebo>
 </robot>
