Commit message: nav2+camera working with preview, snap and face detection not working

File: src/r2d10/urdf/assembly_3.urdf.xacro (robot description, xacro)
@@ -250,5 +250,5 @@
     <link name="camera_link">
     <inertial>
-      <origin xyz="0 0 0" rpy="0 0 0"/>
+      <origin xyz="0 0 0" rpy="0 0 -1.57"/>
       <mass value="0.1"/>
       <inertia ixx="1e-4" iyy="1e-4" izz="1e-4" ixy="0" iyz="0" ixz="0"/>

Commit message: camera fixed and images being saved

File: src/r2d10/urdf/assembly_3.urdf.xacro (robot description, xacro)
@@ -271,5 +271,5 @@
     <parent link="chassis"/>
     <child link="camera_link"/>
-    <origin xyz="0 0 0.12" rpy="0 0 0"/>
+    <origin xyz="0 0 0.12" rpy="0 0 1.57"/>
   </joint>
     <gazebo reference="camera_link">
@@ -278,5 +278,5 @@
       <update_rate>10</update_rate>
       <visualize>true</visualize>
-      <topic>camera</topic>  <!-- Changed from /camera/image_raw -->
+      <topic>/camera/image</topic>
       <camera>
         <horizontal_fov>1.047</horizontal_fov>
